Commit message: first commit

File: catkinws/src/my_robot/urdf/my_robot.xacro (robot description, xacro)
@@ -1,4 +1,5 @@
 <?xml version='1.0'?>
-<robot name="my_robot" xmlns:xacro="http://www.ros.org/wiki/xacro">
+<robot name="my_robot" xmlns:xacro="http://ros.org/wiki/xacro">
+<xacro:include filename="$(find my_robot)/urdf/my_robot.gazebo"/>
                                                   <link name="robot_footprint"></link>
                                                   <joint name="robot_footprint_joint" type="fixed">
@@ -113,3 +114,164 @@
     <dynamics damping="1.0" friction="1.0"/>
   </joint>
+  <!-- Camera Link -->
+<link name="camera">
+  <visual>
+    <origin xyz="0 0 0" rpy="0 0 0"/>
+    <geometry>
+      <box size="0.05 0.05 0.05"/>
+    </geometry>
+  </visual>
+  <collision>
+    <origin xyz="0 0 0" rpy="0 0 0"/>
+    <geometry>
+      <box size="0.05 0.05 0.05"/>
+    </geometry>
+  </collision>
+  <inertial>
+    <origin xyz="0 0 0" rpy="0 0 0"/>
+    <mass value="0.1"/>
+    <inertia
+      ixx="1e-6"
+      ixy="0"
+      ixz="0"
+      iyy="1e-6"
+      iyz="0"
+      izz="1e-6"/>
+  </inertial>
+</link>
+<!-- Camera Joint -->
+<joint name="camera_joint" type="fixed">
+  <parent link="chassis"/>
+  <child link="camera"/>
+  <origin xyz="0.2 0 0" rpy="0 0 0"/>
+  <axis xyz="0 1 0"/>
+</joint>
+<!-- Hokuyo Lidar Link -->
+<link name="hokuyo">
+  <visual>
+    <origin xyz="0 0 0" rpy="0 0 0"/>
+    <geometry>
+      <mesh filename="package://my_robot/meshes/hokuyo.dae"/>
+    </geometry>
+  </visual>
+  <collision>
+    <origin xyz="0 0 0" rpy="0 0 0"/>
+    <geometry>
+      <box size="0.1 0.1 0.1"/>
+    </geometry>
+  </collision>
+  <inertial>
+    <origin xyz="0 0 0" rpy="0 0 0"/>
+    <mass value="1e-5"/>
+    <inertia
+      ixx="1e-6"
+      ixy="0"
+      ixz="0"
+      iyy="1e-6"
+      iyz="0"
+      izz="1e-6"/>
+  </inertial>
+</link>
+<!-- Hokuyo Joint -->
+<joint name="hokuyo_joint" type="fixed">
+  <parent link="chassis"/>
+  <child link="hokuyo"/>
+  <origin xyz="0.15 0 0.1" rpy="0 0 0"/>
+  <axis xyz="0 1 0"/>
+</joint>
+<gazebo>
+    <plugin name="differential_drive_controller" filename="libgazebo_ros_diff_drive.so">
+      <legacyMode>false</legacyMode>
+      <alwaysOn>true</alwaysOn>
+      <updateRate>10</updateRate>
+      <leftJoint>left_wheel_hinge</leftJoint>
+      <rightJoint>right_wheel_hinge</rightJoint>
+      <wheelSeparation>0.4</wheelSeparation>
+      <wheelDiameter>0.2</wheelDiameter>
+      <torque>10</torque>
+      <commandTopic>cmd_vel</commandTopic>
+      <odometryTopic>odom</odometryTopic>
+      <odometryFrame>odom</odometryFrame>
+      <robotBaseFrame>robot_footprint</robotBaseFrame>
+      <publishWheelTF>false</publishWheelTF>
+      <publishWheelJointState>false</publishWheelJointState>
+      <rosDebugLevel>na</rosDebugLevel>
+      <wheelAcceleration>0</wheelAcceleration>
+      <wheelTorque>5</wheelTorque>
+      <odometrySource>world</odometrySource>
+      <publishTf>1</publishTf>
+      <publishOdomTF>true</publishOdomTF>
+    </plugin>
+  </gazebo>
+  <!-- camera -->
+  <gazebo reference="camera">
+    <sensor type="camera" name="camera1">
+      <update_rate>30.0</update_rate>
+      <camera name="head">
+        <horizontal_fov>1.3962634</horizontal_fov>
+        <image>
+          <width>800</width>
+          <height>800</height>
+          <format>R8G8B8</format>
+        </image>
+        <clip>
+          <near>0.02</near>
+          <far>300</far>
+        </clip>
+      </camera>
+      <plugin name="camera_controller" filename="libgazebo_ros_camera.so">
+        <alwaysOn>true</alwaysOn>
+        <updateRate>0.0</updateRate>
+        <cameraName>camera</cameraName>
+        <imageTopicName>rgb/image_raw</imageTopicName>
+        <cameraInfoTopicName>rgb/camera_info</cameraInfoTopicName>
+        <frameName>camera</frameName>
+        <hackBaseline>0.07</hackBaseline>
+        <distortionK1>0.0</distortionK1>
+        <distortionK2>0.0</distortionK2>
+        <distortionK3>0.0</distortionK3>
+        <distortionT1>0.0</distortionT1>
+        <distortionT2>0.0</distortionT2>
+      </plugin>
+    </sensor>
+  </gazebo>
+  <!-- hokuyo -->
+  <gazebo reference="hokuyo">
+    <sensor type="ray" name="head_hokuyo_sensor">
+      <pose>0 0 0 0 0 0</pose>
+      <visualize>false</visualize>
+      <update_rate>40</update_rate>
+      <ray>
+        <scan>
+          <horizontal>
+            <samples>720</samples>
+            <resolution>1</resolution>
+            <min_angle>-1.570796</min_angle>
+            <max_angle>1.570796</max_angle>
+          </horizontal>
+        </scan>
+        <range>
+          <min>0.10</min>
+          <max>30.0</max>
+          <resolution>0.01</resolution>
+        </range>
+        <noise>
+          <type>gaussian</type>
+          <!-- Noise parameters based on published spec for Hokuyo laser
+               achieving "+-30mm" accuracy at range < 10m.  A mean of 0.0m and
+               stddev of 0.01m will put 99.7% of samples within 0.03m of the true
+               reading. -->
+          <mean>0.0</mean>
+          <stddev>0.01</stddev>
+        </noise>
+      </ray>
+      <plugin name="gazebo_ros_head_hokuyo_controller" filename="libgazebo_ros_laser.so">
+        <topicName>/scan</topicName>
+        <frameName>hokuyo</frameName>
+      </plugin>
+    </sensor>
+  </gazebo>
+<commandTopic>cmd_vel</commandTopic>
+<imageTopicName>rgb/image_raw</imageTopicName>
+<topicName>/scan</topicName>
 </robot>

Commit message: first commit

File: catkinws/src/my_robot/urdf/my_robot.xacro (robot description, xacro)
@@ -2,58 +2,66 @@
 <robot name="my_robot" xmlns:xacro="http://ros.org/wiki/xacro">
 <xacro:include filename="$(find my_robot)/urdf/my_robot.gazebo"/>
-                                                  <link name="robot_footprint"></link>
-                                                  <joint name="robot_footprint_joint" type="fixed">
-                                                    <origin xyz="0 0 0" rpy="0 0 0" />
-                                                    <parent link="robot_footprint"/>
-                                                    <child link="chassis" />
-                                                  </joint>
-                                                  <link name='chassis'>
-                                                    <pose>0 0 0.1 0 0 0</pose>
-                                                    <inertial>
-                                                      <mass value="15.0"/>
-                                                      <origin xyz="0.0 0 0" rpy=" 0 0 0"/>
-                                                      <inertia
-                                                          ixx="0.1" ixy="0" ixz="0"
-                                                          iyy="0.1" iyz="0"
-                                                          izz="0.1"
-                                                      />
-                                                    </inertial>
-                                                    <collision name='collision'>
-                                                      <origin xyz="0 0 0" rpy=" 0 0 0"/>
-                                                      <geometry>
-                                                        <box size=".4 .2 .1"/>
-                                                      </geometry>
-                                                    </collision>
-                                                    <visual name='chassis_visual'>
-                                                      <origin xyz="0 0 0" rpy=" 0 0 0"/>
-                                                      <geometry>
-                                                        <box size=".4 .2 .1"/>
-                                                      </geometry>
-                                                    </visual>
-                                                    <collision name='back_caster_collision'>
-                                                      <origin xyz="-0.15 0 -0.05" rpy=" 0 0 0"/>
-                                                      <geometry>
-                                                        <sphere radius="0.0499"/>
-                                                      </geometry>
-                                                    </collision>
-                                                    <visual name='back_caster_visual'>
-                                                      <origin xyz="-0.15 0 -0.05" rpy=" 0 0 0"/>
-                                                      <geometry>
-                                                        <sphere radius="0.05"/>
-                                                      </geometry>
-                                                    </visual>
-                                                    <collision name='front_caster_collision'>
-                                                      <origin xyz="0.15 0 -0.05" rpy=" 0 0 0"/>
-                                                      <geometry>
-                                                        <sphere radius="0.0499"/>
-                                                      </geometry>
-                                                    </collision>
-                                                    <visual name='front_caster_visual'>
-                                                      <origin xyz="0.15 0 -0.05" rpy=" 0 0 0"/>
-                                                      <geometry>
-                                                        <sphere radius="0.05"/>
-                                                      </geometry>
-                                                    </visual>
-                                                  </link>
+<link name="robot_footprint"></link>
+<joint name="robot_footprint_joint" type="fixed">
+               <origin xyz="0 0 0" rpy="0 0 0" />
+               <parent link="robot_footprint"/>
+               <child link="chassis" />
+</joint>
+<link name='chassis'>
+      <pose>0 0 0.1 0 0 0</pose>
+      <inertial>
+      <mass value="15.0"/>
+      <origin xyz="0.0 0 0" rpy=" 0 0 0"/>
+      <inertia
+        ixx="0.1" ixy="0" ixz="0"
+        iyy="0.1" iyz="0"
+        izz="0.1"/>
+</inertial>
+<collision name='collision'>
+      <origin xyz="0 0 0" rpy=" 0 0 0"/>
+      <geometry>
+          <box size="0.5 0.4 0.1"/>
+      </geometry>
+</collision>
+<visual name='chassis_visual'>
+      <origin xyz="0 0 0" rpy=" 0 0 0"/>
+      <geometry>
+           <box size="0.5 0.4 0.1"/>
+      </geometry>
+      <material name="silver">
+        <color rgba="0.75 0.75 0.75 1"/>
+      </material>
+</visual>
+<collision name='back_caster_collision'>
+      <origin xyz="-0.15 0 -0.05" rpy=" 0 0 0"/>
+      <geometry>
+            <sphere radius="0.0499"/>
+      </geometry>
+</collision>
+<visual name='back_caster_visual'>
+      <origin xyz="-0.15 0 -0.05" rpy=" 0 0 0"/>
+      <geometry>
+             <sphere radius="0.05"/>
+      </geometry>
+      <material name="red">
+        <color rgba="1 0 0 1"/>
+      </material>
+</visual>
+<collision name='front_caster_collision'>
+      <origin xyz="0.15 0 -0.05" rpy=" 0 0 0"/>
+      <geometry>
+         <sphere radius="0.0499"/>
+      </geometry>
+</collision>
+<visual name='front_caster_visual'>
+                    <origin xyz="0.15 0 -0.05" rpy=" 0 0 0"/>
+                    <geometry>
+                          <sphere radius="0.05"/>
+                    </geometry>
+      <material name="red">
+        <color rgba="1 0 0 1"/>
+      </material>
+</visual>
+ </link>
 <!-- Left Wheel -->
 <link name="left_wheel">
@@ -66,12 +74,14 @@
     <origin xyz="0 0 0" rpy="0 1.5707 1.5707"/>
     <geometry>
-      <cylinder radius="0.1" length="0.05"/>
-    </geometry>
-    <material name="black"/>
-  </visual>
-  <collision>
-    <origin xyz="0 0 0" rpy="0 1.5707 1.5707"/>
-    <geometry>
-      <cylinder radius="0.1" length="0.05"/>
+      <cylinder radius="0.2" length="0.1"/>
+    </geometry>
+    <material name="black">
+      <color rgba="0 0 0 1"/>
+    </material>
+  </visual>
+  <collision>
+    <origin xyz="0 0 0" rpy="0 1.5707 1.5707"/>
+    <geometry>
+      <cylinder radius="0.2" length="0.1"/>
     </geometry>
   </collision>
@@ -87,12 +97,14 @@
     <origin xyz="0 0 0" rpy="0 1.5707 1.5707"/>
     <geometry>
-      <cylinder radius="0.1" length="0.05"/>
-    </geometry>
-    <material name="black"/>
-  </visual>
-  <collision>
-    <origin xyz="0 0 0" rpy="0 1.5707 1.5707"/>
-    <geometry>
-      <cylinder radius="0.1" length="0.05"/>
+      <cylinder radius="0.2" length="0.1"/>
+    </geometry>
+    <material name="black">
+      <color rgba="0 0 0 1"/>
+    </material>
+  </visual>
+  <collision>
+    <origin xyz="0 0 0" rpy="0 1.5707 1.5707"/>
+    <geometry>
+      <cylinder radius="0.2" length="0.1"/>
     </geometry>
   </collision>
